File: schematics_pcb/internal-pontag/pontag.kicad_pcb (KiCad board)
At the start: 2 copper layers, 31 parts, among them J1 PWR Connector, J2 Floppy PWR Connector, J3 RS232 Port, J4 PS/2 Mouse, J5 AVR-ISP-6, J7 Extra, SW1 Reset, U1 L78L05_TO92, U3 ATmega328P-PU, U4 MAX232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

Commit message: prepare files for internal PCB
Parts:
- C5, C6: footprint Capacitor_THT:C_Disc_D3.4mm_W2.1mm_P2.50mm -> Capacitor_THT:C_Disc_D4.3mm_W1.9mm_P5.00mm
